File: Kicad/cap-locator/cap-locator.kicad_pcb (KiCad board)
At the start: 2 copper layers, 20 parts, among them J1 Conn_01x02, J2 Conn_01x05, J3 Conn_01x02, J4 Conn_01x02, J5 Conn_01x02, J6 Conn_01x02, J7 USB_B_Micro, J8 Conn_01x03, U1 PIC16F1455-IST

Commit message: 回路図記載
Parts:
- removed J2: Conn_01x05, Connector_JST:JST_EH_B5B-EH-A_1x05_P2.50mm_Vertical
- added D1: LED, LED_SMD:LED_0603_1608Metric, F.Cu at (154.8, 67.3)
- added D3: LED, LED_SMD:LED_0603_1608Metric, F.Cu at (171.9, 81.2)
- added D4: LED, LED_SMD:LED_0603_1608Metric, F.Cu at (171.9, 83.8)
- added D5: LED, LED_SMD:LED_0603_1608Metric, F.Cu at (171.9, 86.4)
- added J9: Writer, Connector_PinSocket_2.00mm:PinSocket_1x06_P2.00mm_Horizontal, F.Cu at (167.9, 81.9)
- added R7: 470R, Resistor_SMD:R_0603_1608Metric, F.Cu at (154.8, 69.8)
- C1, C2: value C -> 0.1uf; footprint Capacitor_SMD:C_0805_2012Metric -> Capacitor_SMD:C_0603_1608Metric
- D1, D2: footprint LED_SMD:LED_1206_3216Metric -> LED_SMD:LED_0603_1608Metric
- J8: value Conn_01x03 -> CH213K
- R1: value R -> 10K; footprint Resistor_SMD:R_0805_2012Metric -> Resistor_SMD:R_0603_1608Metric
- R2, R3, R4, R5, R6: value R -> 470R; footprint Resistor_SMD:R_0805_2012Metric -> Resistor_SMD:R_0603_1608Metric
Connections:
- C1 pad 1: unconnected-(C1-Pad1) -> GND
- C1 pad 2: unconnected-(C1-Pad2) -> VCC
- C2 pad 1: unconnected-(C2-Pad1) -> GND
- C2 pad 2: unconnected-(C2-Pad2) -> Net-(U1-Vusb3v3)
- D1 pad 1: unconnected-(D1-K-Pad1) -> GND
- D1 pad 2: unconnected-(D1-A-Pad2) -> Net-(D1-A)
- D2 pad 1: unconnected-(D2-K-Pad1) -> GND
- D2 pad 2: unconnected-(D2-A-Pad2) -> Net-(D2-A)
- J1 pad 1: unconnected-(J1-Pin_1-Pad1) -> Net-(J1-Pin_1)
- J1 pad 2: unconnected-(J1-Pin_2-Pad2) -> GND
- J3 pad 1: unconnected-(J3-Pin_1-Pad1) -> Net-(J3-Pin_1)
- J3 pad 2: unconnected-(J3-Pin_2-Pad2) -> GND
- J4 pad 1: unconnected-(J4-Pin_1-Pad1) -> Net-(J4-Pin_1)
- J4 pad 2: unconnected-(J4-Pin_2-Pad2) -> GND
- J5 pad 1: unconnected-(J5-Pin_1-Pad1) -> Net-(J5-Pin_1)
- J5 pad 2: unconnected-(J5-Pin_2-Pad2) -> GND
- J6 pad 1: unconnected-(J6-Pin_1-Pad1) -> Net-(J6-Pin_1)
- J6 pad 2: unconnected-(J6-Pin_2-Pad2) -> GND
- J7 pad 1: unconnected-(J7-VBUS-Pad1) -> Net-(J7-VBUS)
- J7 pad 2: unconnected-(J7-D--Pad2) -> D-
- J7 pad 3: unconnected-(J7-D+-Pad3) -> D+
- J8 pad 1: unconnected-(J8-Pin_1-Pad1) -> GND
- J8 pad 2: unconnected-(J8-Pin_2-Pad2) -> VCC
- J8 pad 3: unconnected-(J8-Pin_3-Pad3) -> Net-(J7-VBUS)
- R1 pad 1: unconnected-(R1-Pad1) -> MCLR
- R1 pad 2: unconnected-(R1-Pad2) -> VCC
- R2 pad 1: unconnected-(R2-Pad1) -> Net-(J1-Pin_1)
- R2 pad 2: unconnected-(R2-Pad2) -> Location1
- R3 pad 1: unconnected-(R3-Pad1) -> Net-(J3-Pin_1)
- R3 pad 2: unconnected-(R3-Pad2) -> Location2
- R4 pad 1: unconnected-(R4-Pad1) -> Net-(J4-Pin_1)
- R4 pad 2: unconnected-(R4-Pad2) -> Location3
- R5 pad 1: unconnected-(R5-Pad1) -> Net-(J5-Pin_1)
- R5 pad 2: unconnected-(R5-Pad2) -> Location4
- R6 pad 1: unconnected-(R6-Pad1) -> Net-(J6-Pin_1)
- R6 pad 2: unconnected-(R6-Pad2) -> Location5
- U1 pad 1: unconnected-(U1-VDD-Pad1) -> VCC
- U1 pad 10: unconnected-(U1-ICSPDAT/SCK/SCL/C2IN+/C1IN+/Vref+/AN4/RC0-Pad10) -> ICSPDAT
- U1 pad 11: unconnected-(U1-Vusb3v3-Pad11) -> Net-(U1-Vusb3v3)
- U1 pad 12: unconnected-(U1-RA1/D-/ICSPCLK-Pad12) -> D-
- U1 pad 13: unconnected-(U1-RA0/D+/ICSPDAT-Pad13) -> D+
- U1 pad 14: unconnected-(U1-VSS-Pad14) -> GND
- U1 pad 2: unconnected-(U1-RA5/SOSCI/T1CKI/PWM2/CLKIN/OSC1-Pad2) -> Net-(U1-RA5/SOSCI/T1CKI/PWM2/CLKIN/OSC1)
- U1 pad 3: unconnected-(U1-RA4/AN3/SOSCO/T1G/SDO/CLKOUT/OSC2/CLKR-Pad3) -> Location5
- U1 pad 4: unconnected-(U1-RA3/T1G/~{SS}/~{MCLR}/Vpp-Pad4) -> MCLR
- U1 pad 5: unconnected-(U1-PWM1/DT/RX/CWG1A/T0CKI/RC5-Pad5) -> Location4
- U1 pad 6: unconnected-(U1-CK/TX/CWG1B/C1OUT/C2OUT/RC4-Pad6) -> Location3
- U1 pad 7: unconnected-(U1-CLKR/~{SS}/PWM2/C1IN3-/C2IN3-/DACOUT2/AN7/RC3-Pad7) -> Location2
- U1 pad 8: unconnected-(U1-SDO/C2IN2-/C1IN2-/DACOUT1/AN6/RC2-Pad8) -> Location1
- U1 pad 9: unconnected-(U1-ICSPCLK/SDI/SDA/~{CWGFLT}/C2IN-/C1IN-/AN5/RC1-Pad9) -> ICSPCLK

Commit message: 基板発注
Parts:
- removed C3: C, Capacitor_SMD:C_0805_2012Metric
- removed the D1 at (154.8, 67.3)
- removed the D1 at (148.6, 82.5)
- removed D2, D3, D4, D5: LED, LED_SMD:LED_0603_1608Metric
- added D1: LED, LED_SMD:LED_0603_1608Metric, F.Cu at (152.2, 108.4)
- added MH1: MountingHole_3.2mm_M3, MountingHole:MountingHole_3.2mm_M3, F.Cu at (135.0, 125.0)
- added MH2: MountingHole_3.2mm_M3, MountingHole:MountingHole_3.2mm_M3, F.Cu at (152.0, 79.0)
- added U2: USBLC6-2SC6, Package_TO_SOT_SMD:SOT-23-6, F.Cu at (144.8, 120.5)
- C2: value 0.1uf -> 1uf
- U1: footprint Package_SO:SOIC-14W_7.5x9mm_P1.27mm -> Package_SO:TSSOP-14_4.4x5mm_P0.65mm
- moved R3 50.1 mm to (141.4, 108.4)
- moved R2 49.1 mm to (141.4, 117.3)
- moved J3 38.6 mm to (137.5, 108.2)
- moved J1 37.0 mm to (137.5, 117.2)
- moved R7 36.7 mm to (152.2, 106.5)
- moved J5 31.5 mm to (137.5, 90.2)
- moved C2 30.8 mm to (154.1, 100.8), turned to -90 degrees
- moved J8 28.0 mm to (149.4, 121.6), turned to -90 degrees
- moved J6 27.5 mm to (137.5, 81.2)
- moved J7 24.1 mm to (144.4, 126.4)
- moved J9 23.6 mm to (148.3, 95.0), turned to 180 degrees
- moved R1 20.6 mm to (144.2, 94.1), turned to 90 degrees
- moved U1 19.3 mm to (149.1, 102.1)
- moved R6 16.7 mm to (141.4, 81.1)
- moved R5 16.2 mm to (141.4, 90.0)
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Connections:
- J7 pad 2: D- -> Net-(J7-D-)
- J7 pad 3: D+ -> Net-(J7-D+)
- J7 pad 5: unconnected-(J7-GND-Pad5) -> GND
Routing:
- net VCC: track 0.00 -> 60.5 mm, vias 0 -> 2
- net Location5: track 0.00 -> 23.4 mm, vias 0 -> 2
- net D+: track 0.00 -> 23.3 mm, vias 0 -> 2
- net D-: track 0.00 -> 21.5 mm, vias 0 -> 2
- net ICSPCLK: track 0.00 -> 21.1 mm, vias 0 -> 2
- net Location1: track 0.00 -> 17.9 mm
- net ICSPDAT: track 0.00 -> 16.4 mm, vias 0 -> 2
- net GND: track 0.00 -> 16.2 mm, vias 0 -> 28
- net Location4: track 0.00 -> 14.8 mm
- net MCLR: track 0.00 -> 13.4 mm
- net Net-(J7-D+): track 0.00 -> 11.2 mm
- net Net-(U1-RA5/SOSCI/T1CKI/PWM2/CLKIN/OSC1): track 0.00 -> 9.14 mm, vias 0 -> 2
- net Net-(J7-VBUS): track 0.00 -> 7.74 mm, vias 0 -> 2
- net Location2: track 0.00 -> 6.03 mm
- net Location3: track 0.00 -> 5.82 mm
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- added copper zone on B.Cu, net GND
- added copper zone on F.Cu, net GND
Other:
- board outline added: 26.9 x 56 mm
- board text added: "cap-locator.1.0.0 2025/11/17"
