File: Kicad/cap-locator/cap-locator.kicad_sch (KiCad schematic)
At the start: 20 parts, among them J1 Conn_01x02, J2 Conn_01x05, J3 Conn_01x02, J4 Conn_01x02, J5 Conn_01x02, J6 Conn_01x02, J7 USB_B_Micro, J8 Conn_01x03, U1 PIC16F1455-IST

Commit message: 回路図記載
Parts:
- removed C3: C, Capacitor_SMD:C_0805_2012Metric, symbol Device:C
- removed D2: LED, LED_SMD:LED_1206_3216Metric, symbol Device:LED
- removed J2: Conn_01x05, Connector_JST:JST_EH_B5B-EH-A_1x05_P2.50mm_Vertical, symbol Connector_Generic:Conn_01x05
- added J9: Writer, Connector_PinSocket_2.00mm:PinSocket_1x06_P2.00mm_Horizontal, symbol Connector_Generic:Conn_01x06
- added R7: 470R, Resistor_SMD:R_0603_1608Metric, symbol Device:R
- C1, C2: value C -> 0.1uf; footprint Capacitor_SMD:C_0805_2012Metric -> Capacitor_SMD:C_0603_1608Metric
- D1: footprint LED_SMD:LED_1206_3216Metric -> LED_SMD:LED_0603_1608Metric
- J8: value Conn_01x03 -> CH213K
- R1: value R -> 10K; footprint Resistor_SMD:R_0805_2012Metric -> Resistor_SMD:R_0603_1608Metric
- R2, R3, R4, R5, R6: value R -> 470R; footprint Resistor_SMD:R_0805_2012Metric -> Resistor_SMD:R_0603_1608Metric
Connections:
- net at J7.1 (VBUS): now also J8.3 (Pin_3)
- net D-: now reaches J7.2 (D-)
- net D-: now also U1.12 (RA1/D-/ICSPCLK)
- net D+: now reaches J7.3 (D+)
- net D+: now also U1.13 (RA0/D+/ICSPDAT)
- net VCC: now reaches U1.1 (VDD)
- net VCC: now also C1.2, J8.2 (Pin_2), R1.2, J9.2 (Pin_2)
- net ICSPDAT: now reaches U1.10 (ICSPDAT/SCK/SCL/C2IN+/C1IN+/Vref+/AN4/RC0)
- net ICSPDAT: now also J9.4 (Pin_4)
- net at U1.11 (Vusb3v3): now also C2.2
- net GND: now reaches U1.14 (VSS)
- net GND: now also C1.1, C2.1, D1.1 (K), J1.2 (Pin_2), J3.2 (Pin_2), J4.2 (Pin_2), J5.2 (Pin_2), J6.2 (Pin_2), J8.1 (Pin_1), J9.3 (Pin_3)
- net at U1.2 (RA5/SOSCI/T1CKI/PWM2/CLKIN/OSC1): now also R7.1
- net Location5: now reaches U1.3 (RA4/AN3/SOSCO/T1G/SDO/CLKOUT/OSC2/CLKR)
- net Location5: now also R6.2
- net MCLR: now reaches U1.4 (RA3/T1G/~{SS}/~{MCLR}/Vpp)
- net MCLR: now also R1.1, J9.1 (Pin_1)
- net Location4: now reaches U1.5 (PWM1/DT/RX/CWG1A/T0CKI/RC5)
- net Location4: now also R5.2
- net Location3: now reaches U1.6 (CK/TX/CWG1B/C1OUT/C2OUT/RC4)
- net Location3: now also R4.2
- net Location2: now reaches U1.7 (CLKR/~{SS}/PWM2/C1IN3-/C2IN3-/DACOUT2/AN7/RC3)
- net Location2: now also R3.2
- net Location1: now reaches U1.8 (SDO/C2IN2-/C1IN2-/DACOUT1/AN6/RC2)
- net Location1: now also R2.2
- net ICSPCLK: now reaches U1.9 (ICSPCLK/SDI/SDA/~{CWGFLT}/C2IN-/C1IN-/AN5/RC1)
- net ICSPCLK: now also J9.5 (Pin_5)
- net at R3.1: now also J3.1 (Pin_1)
- net at R6.1: now also J6.1 (Pin_1)
- net at R2.1: now also J1.1 (Pin_1)
- net at J4.1 (Pin_1): now also R4.1
- net at J5.1 (Pin_1): now also R5.1
- net at D1.2 (A): now also R7.2
- no-connect marks 0 -> 4
Other:
- moved on the sheet: C1, C2, J1, J3, J4, J5, J6, J7, R1, R2, R3, R4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

Commit message: 基板発注
Parts:
- added U2: USBLC6-2SC6, Package_TO_SOT_SMD:SOT-23-6, symbol Power_Protection:USBLC6-2SC6
- C2: value 0.1uf -> 1uf
- U1: footprint Package_SO:SOIC-14W_7.5x9mm_P1.27mm -> Package_SO:TSSOP-14_4.4x5mm_P0.65mm
Connections:
- net D+: now also U2.6 (I/O1); no longer J7.3 (D+)
- net D-: now also U2.4 (I/O2); no longer J7.2 (D-)
- net GND: now also J7.5 (GND), U2.2 (GND)
- net VCC: now also U2.5 (VBUS)
- new net: J7.2 (D-), U2.3 (I/O2)
- new net: J7.3 (D+), U2.1 (I/O1)
- no-connect marks 4 -> 3
Other:
- company: (none) -> GTech
- title: (none) -> cap-locator
- moved on the sheet: J8
